File: BMW_E30_Gauge_Cluster_Early_Model/BMW_E30_Early_Cluster_Nexus/BMW_E30_Early_Cluster_Nexus.kicad_sch (KiCad schematic)
At the start: 26 parts, among them J1 C1 - Blue Connector, J2 C2 - White Connector, J3 C3 - Yellow Connector, J4 Conn_01x16_Pin, J5 Conn_01x19_Socket, U1 Temperature Gauge, U2 Fuel Gauge

Commit message: Layout Updates
Layout traces completed. All footprints are also in now and lined up with the scan. Still need to fix illum and charge indicator conflict on the right side of the board.
Parts:
- J4: footprint (none) -> BMW_Cluster_Connectors:ConnectorIV_Early
- J5: footprint (none) -> BMW_Cluster_Connectors:ConnectorV_Early
- U1, U2: footprint (none) -> BMW_Cluster_Connectors:Gauge_fuel_temp
Changed lines of the file:
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@@
 			)
 		)
-		(property "Footprint" ""
+		(property "Footprint" "BMW_Cluster_Connectors:ConnectorIV_Early"
 			(at 101.6 116.84 0)
 			(effects
@@
 			)
 		)
-		(property "Footprint" ""
+		(property "Footprint" "BMW_Cluster_Connectors:Gauge_fuel_temp"
 			(at 127 207.01 0)
 			(effects
@@
 			)
 		)
-		(property "Footprint" ""
+		(property "Footprint" "BMW_Cluster_Connectors:ConnectorV_Early"
 			(at 29.21 121.92 0)
 			(effects
@@
 			)
 		)
-		(property "Footprint" ""
+		(property "Footprint" "BMW_Cluster_Connectors:Gauge_fuel_temp"
 			(at 227.33 205.74 0)
 			(effects

Commit message: Layout Update
Added in resistor parallel to the charge indicator light. This will prevent the alternator from not charging in the event that the charge indicator bulb burns out.
Parts:
- R4: value 51R -> 100R; footprint Resistor_THT:R_Axial_DIN0516_L15.5mm_D5.0mm_P20.32mm_Horizontal -> Resistor_THT:R_Axial_DIN0414_L11.9mm_D4.5mm_P15.24mm_Horizontal; now fitted
Changed lines of the file:
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@@
 		(in_bom yes)
 		(on_board yes)
-		(dnp yes)
+		(dnp no)
 		(fields_autoplaced yes)
 		(property "Reference" "R4"
@@
 			)
 		)
-		(property "Value" "51R"
+		(property "Value" "100R"
 			(at 325.12 123.1899 0)
 			(effects
@@
 			)
 		)
-		(property "Footprint" "Resistor_THT:R_Axial_DIN0516_L15.5mm_D5.0mm_P20.32mm_Horizontal"
+		(property "Footprint" "Resistor_THT:R_Axial_DIN0414_L11.9mm_D4.5mm_P15.24mm_Horizontal"
 			(at 320.802 121.92 90)
 			(effects

Commit message: Added SI Bypass
Added in jumper pads that allow the SI board to be fully removed while maintaining functionality of the temperature gauge which would otherwise be disconnected.

Idea by user: mayacaine
Edited and merged by: Ansel84
Parts:
- added JP1: SI BYPASS, Jumper:SolderJumper-2_P1.3mm_Open_RoundedPad1.0x1.5mm, symbol Jumper:SolderJumper_2_Open
Connections:
- net Eng_temp_sensor: now also JP1.2 (B)
- net Temp_gauge: now also JP1.1 (A)
Other:
- note added: "SI Board Connector"
- note added: "SI Bypass Option"
- moved on the sheet: LA12, LA14, R2, R3, U1, U2
